File: lite/hardware/kicad/Linetracer2-Lite.kicad_pcb (KiCad board)
At the start: 2 copper layers, 65 x 100 mm, 36 parts, among them J1 BATTERY (AA x3, XH 2P), M1 LEFT motor FA-130RA, M2 RIGHT motor FA-130RA, Q1 2SC1815-GR, SW1 START, U1 XIAO ESP32C6, U2 AE-TC78H653FTG

Commit message: Lite: フルカラー LED を 6 こ・左右の端に、流れる光、テストパッド
- PL9823 ×6（D2〜D7）を基板の左右の端に 3 こずつ縦に。信号は D6 → 左のうしろ → 左の前 →
  前の端をわたって → 右の前 → 右のうしろ。電源 VSYS は裏の線（右の列の内側 → 前を横切って → 左の列の内側）
- 場所をあけるため Q1 を R7 の前へ（180° 回転）、抵抗の絵を真ん中へ、S3 の線を内側へ。C5 はなくした
- テストパッド 7 こ（GND・3V3・VSYS・S1・S2・S3・IR、表の SMD）＋ D1 の上のパッドに VBAT。
  値の表（README §4.9）と先生用プログラム 08_test_pads.py
- ソフト: robot.led.flow(左, 右) = 両側で光が前→うしろへ、その側の車輪の速さで流れる（走っているとき）。
  side() / count() / bar() も 6 こ用に。サンプル 07_rgb_led.py を直した
- DRC / ERC 0、ビア 0、干渉チェックはすべて空。手順の絵・3D・Gerber・部品表（1 台 約 ¥2,760）を作り直した

Co-Authored-By: Claude Opus 5.5 <noreply@anthropic.com>
Parts:
- removed C5: 0.1uF, Capacitor_THT:C_Disc_D3.0mm_W2.0mm_P2.50mm
- added D7: PL9823, Linetracer2:LED_PL9823_5mm, F.Cu at (179.2, 68.6)
- added TP1: GND, TestPoint:TestPoint_Pad_D1.5mm, F.Cu at (150.0, 72.6)
- added TP2: 3V3, TestPoint:TestPoint_Pad_D1.5mm, F.Cu at (150.0, 68.2)
- added TP3: VSYS, TestPoint:TestPoint_Pad_D1.5mm, F.Cu at (181.0, 91.5)
- added TP4: SENS1, TestPoint:TestPoint_Pad_D1.5mm, F.Cu at (147.2, 66.6)
- added TP5: SENS2, TestPoint:TestPoint_Pad_D1.5mm, F.Cu at (159.0, 65.3)
- added TP6: SENS3, TestPoint:TestPoint_Pad_D1.5mm, F.Cu at (171.0, 64.0)
- added TP7: LED_K, TestPoint:TestPoint_Pad_D1.5mm, F.Cu at (128.8, 57.8)
- moved D6 43.0 mm to (179.2, 61.6), turned to -90 degrees
- moved D5 41.8 mm to (179.2, 54.6), turned to -90 degrees
- moved D4 39.3 mm to (120.8, 54.6), turned to 90 degrees
- moved D3 29.6 mm to (120.8, 61.6), turned to 90 degrees
- moved D2 20.1 mm to (120.8, 68.6), turned to 90 degrees
- moved Q1 10.2 mm to (130.7, 53.2), turned to 180 degrees
Connections:
- D6 pad 2: unconnected-(D6-DO-Pad2) -> Net-(D6-DO)
Routing:
- net Net-(D4-DO): track 8.45 -> 61.0 mm
- net /VSYS: track 95.6 -> 129.1 mm
- net /RGB_DIN: track 31.7 -> 45.5 mm
- net Net-(D6-DO): track 0.00 -> 3.94 mm
- net Net-(Q1-B): track 3.50 -> 4.80 mm
- net /LED_K: track 42.1 -> 43.2 mm
- net /SENS3: track 35.7 -> 34.8 mm
Other:
- board text added: "3V3"
- board text added: "GND"
- board text added: "IR"
- board text added: "Linetracer2"
- board text added: "Lite rev.L3"
- board text added: "VBAT"
- board text added: "VSYS"
- board text removed: "Linetracer2 Lite rev.L3"
