File: lite/hardware/kicad/Linetracer2-Lite.kicad_sch (KiCad schematic)
At the start: 30 parts, among them J1 BATTERY (AA x3, XH 2P), J2 I2C (0.96in OLED order), M1 LEFT motor FA-130RA, M2 RIGHT motor FA-130RA, Q1 2SC1815-GR, SW1 START, U1 Raspberry Pi Pico, U2 AE-TC78H653FTG

Commit message: Lite rev.L3: XIAO（ピンヘッダ）、ブザー、フルカラー LED 6 こ、テストパッド、手で引いた配線、車軸も印刷するギヤボックス (#4)
* Lite rev.L2: XIAO ESP32C6 と LBR-127HLD に変更、子ども向けに配置・シルクを見直し

- マイコンを Seeed Studio XIAO ESP32C6（秋月 129481）に。ピンヘッダなしで基板にじかにはんだ付け
  （自作フットプリント: 裏のテストパッドの下は銅禁止、USB の足の逃げ穴、アンテナの下は両面銅なし）
- フォトリフレクタを LBR-127HLD（秋月 104500）に。背が 5.6 mm あるのでスキッドを 7.5 mm に
  （skid_clip_h70/h75/h80.stl、ロボットは後ろに 2.9° 傾く。傾きとすき間は scad で計算）
- いらない部品: I2C の穴 J2 を削除。電池電圧の測定はなし（XIAO の ADC 3 本をセンサーで使い切る）
- ピン割り当ては ESP32-C6 の起動時の状態に合わせ、どの瞬間もモーターが回らないようにした
- 基板を 65 x 100 mm の長方形に（面積 -27%、3D プリント部品はそのまま）、抵抗を 6 mm おきに
- シルクは記号だけ（つくる順番の数字、＋、LED の絵、抵抗の 3 本目の色）。説明は手順書 lite/docs/assembly.md
- gen_3d.py の 3D モデルの位置ずれを修正（KiCad は VRML の translation に scale をかけない）
- ERC 0、DRC 0（警告 0・未接続 0）。MicroPython (ESP32_GENERIC_C6) のライブラリとサンプルを移植

Co-Authored-By: Claude Opus 5.5 <noreply@anthropic.com>

* Lite の節に、ボールキャスターは標準版用と注記

Co-Authored-By: Claude Opus 5.5 <noreply@anthropic.com>

* Lite 用ボールキャスターを追加し、3D プリント部品を子ども向けに見直した

- Lite 用ボールキャスター caster_lite_print_h70/h75/h80（玉ごと印刷、玉 φ4.0/4.5/5.0）と
  caster_lite_bead_h70/h75/h80（φ4 の玉を押し込む、先生用）。玉はスキッドの穴 (50, 11) のピンの真下。
  玉が重さで押し上げられた状態で、同じ高さのスキッドと同じ傾き・センサーと床のすき間（7.5 mm で 2.9°・2.25 mm）。
  基板設計と決めた範囲（裏 x 45〜55・y 6.5〜16、表 r 2.4）に収め、どの向きに差しても当たらない
- 干渉チェック check_caster_lite_*（sensor / bead_sensor / pcb / ball / bead_ball / floor / ballfloor / zone）と
  check_skidclip_lite_zone を追加（わざとずらした条件で検出することも確認）。-D LITE=true のときは
  check_caster_* が Lite 用キャスターを調べる。assembly は LITE_SUPPORT で skid / caster_print / caster_bead を選べる
- 子ども向け: 枠・デッキ・ツメ版デッキのツメの縦の角を丸め、車輪のふち・ハブを面取り、スキッドの角を丸めた。
  枠に L / R を刻んだ。はまる寸法は変えていない（標準版・Lite とも干渉チェックは全部「空」）
- README に Lite キャスターの節と安全の見直し表、08_knowledge に知見（玉が押し上げられる分、小さい玉ほど
  受けが床に近い、ピニオンの組み立て順の問題）を追記

Co-Authored-By: Claude Opus 5.5 <noreply@anthropic.com>

* Lite rev.L3 基板: XIAO をピンヘッダで、ブザー追加、配線を手で引き直し、シルクを改良

- XIAO ESP32C6 を 2 列 x 7 ピンのスルーホール（ピンヘッダ）に。直付け用フットプリントは削除
- 圧電スピーカー BZ1（PKM13EPYH4000-A0）＋ R9 100 Ω を赤 LED と同じ D6 に
- 自動配線をやめ、lite/scripts/layout_lite.py に配置と配線を書いた（縦・横・45°、直角は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
Parts:
- removed J2: I2C (0.96in OLED order), Connector_PinHeader_2.54mm:PinHeader_1x04_P2.54mm_Vertical, symbol Connector_Generic:Conn_01x04
- removed R8: 1k, Resistor_THT:R_Axial_DIN0207_L6.3mm_D2.5mm_P10.16mm_Horizontal, symbol Device:R
- added BZ1: piezo 13mm, Linetracer2:Buzzer_PKM13_P5.0, symbol Device:Buzzer
- added D3, D4, D5, D6, D7: PL9823, Linetracer2:LED_PL9823_5mm, symbol Linetracer2:PL9823
- added R10: 1k, Resistor_THT:R_Axial_DIN0207_L6.3mm_D2.5mm_P10.16mm_Horizontal, symbol Device:R
- added R9: 100, Resistor_THT:R_Axial_DIN0207_L6.3mm_D2.5mm_P10.16mm_Horizontal, symbol Device:R
- added TP1: GND, TestPoint:TestPoint_Pad_D1.5mm, symbol Connector:TestPoint
- added TP2: 3V3, TestPoint:TestPoint_Pad_D1.5mm, symbol Connector:TestPoint
- added TP3: VSYS, TestPoint:TestPoint_Pad_D1.5mm, symbol Connector:TestPoint
- added TP4: SENS1, TestPoint:TestPoint_Pad_D1.5mm, symbol Connector:TestPoint
- added TP5: SENS2, TestPoint:TestPoint_Pad_D1.5mm, symbol Connector:TestPoint
- added TP6: SENS3, TestPoint:TestPoint_Pad_D1.5mm, symbol Connector:TestPoint
- added TP7: LED_K, TestPoint:TestPoint_Pad_D1.5mm, symbol Connector:TestPoint
- C2: Note hold-up for Pico when motors pull the battery down -> hold-up for the XIAO when motors pull the battery down
- D2: value LED red -> PL9823; footprint LED_THT:LED_D3.0mm -> Linetracer2:LED_PL9823_5mm; symbol Device:LED -> Linetracer2:PL9823; Akizuki 111577 -> 108411 (PL9823-F5)
- PS1, PS2, PS3: value LBR-123F -> LBR-127HLD; footprint Linetracer2:LBR-123F -> Linetracer2:LBR-127HLD; symbol Linetracer2:LBR-123F -> Linetracer2:LBR-127HLD; Akizuki 116455 -> 104500
- U1: value Raspberry Pi Pico -> XIAO ESP32C6; footprint Linetracer2:RaspberryPi_Pico_DirectSolder -> Linetracer2:XIAO_ESP32C6_Header; symbol Linetracer2:RaspberryPi_Pico_THT -> Linetracer2:XIAO_ESP32C6; Akizuki 116132 (Pico, Pico 2 also OK; not Pico W) -> 129481 (Seeed Studio XIAO ESP32C6) + pin header 1x40 100167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; Note solder the castellated edge straight onto the pads, no pin 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 -> solder the XIAO on two 1x7 pin headers (cut from a 1x40 str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
Connections:
- net I2C_SDA is gone; now on net MOT_IN2: U1.6 (GPIO23/SCL/D5)
- net +3V3: now also U1.12 (3V3), TP2.1; no longer U1.36 (3V3)
- net GND: now also BZ1.2 (-), D3.1 (GND), D4.1 (GND), D5.1 (GND), D6.1 (GND), D7.1 (GND), TP1.1; no longer U1.18 (GND), U1.23 (GND), U1.28 (GND), U1.3 (GND), U1.33 (AGND), U1.38 (GND), U1.8 (GND)
- net LED_K: now also TP7.1
- net MOT_IN1: now also U1.9 (GPIO19/SCK/D8); no longer U1.16 (GPIO12)
- net MOT_IN2: no longer U1.17 (GPIO13)
- net MOT_IN3: now also U1.10 (GPIO20/MISO/D9); no longer U1.19 (GPIO14)
- net MOT_IN4: now also U1.11 (GPIO18/MOSI/D10); no longer U1.20 (GPIO15)
- net MOT_OUT3: now also C4.2, M2.2 (-); no longer C4.1, M2.1 (+)
- net MOT_OUT4: now also C4.1, M2.1 (+); no longer C4.2, M2.2 (-)
- net MOT_STBY: now also U1.8 (GPIO17/RX/D7); no longer U1.15 (GPIO11)
- net SENS1: now also U1.3 (GPIO2/A2/D2), TP4.1; no longer U1.34 (GPIO28_ADC2)
- net SENS2: now also U1.2 (GPIO1/A1/D1), TP5.1; no longer U1.32 (GPIO27_ADC1)
- net SENS3: now also U1.1 (GPIO0/A0/D0), TP6.1; no longer U1.31 (GPIO26_ADC0)
- net SENS_LED_EN: now also U1.4 (GPIO21/D3); no longer U1.2 (GPIO1)
- net SW1: now also U1.5 (GPIO22/SDA/D4), R10.1, R9.1; no longer SW1.1, U1.21 (GPIO16)
- net VSYS: now also D2.3 (VDD), U1.14 (5V), D3.3 (VDD), D4.3 (VDD), D5.3 (VDD), D6.3 (VDD), D7.3 (VDD), TP3.1; no longer U1.39 (VSYS)
- net at D2.2 (DO): now also D3.4 (DIN)
- net I2C_SCL renamed RGB_DIN
- net RGB_DIN: now also D2.4 (DIN)
- removed net LED1: U1.24 (GPIO18)
- new net: BZ1.1 (+), R9.2
- new net: D5.2 (DO), D6.4 (DIN)
- new net: D4.2 (DO), D5.4 (DIN)
- new net: D3.2 (DO), D4.4 (DIN)
- new net: D6.2 (DO), D7.4 (DIN)
- new net BTN: R10.2, SW1.1
- no-connect marks 17 -> 1
Other:
- note added: "(front -> rear). Data from D6 (TX: the boot log may flash them once). 6 x white = 0.36 A: the library limits it."
- note added: "2. MCU Seeed Studio XIAO ESP32C6 (on two 1x7 pin headers)"
- note added: "4. BUTTON / BUZZER / RGB LEDs"
- note added: "5. LINE SENSORS 3 x LBR-127HLD (mount on the BOTTOM side, lens to the floor), 12 mm apart"
- note added: "6. TEST PADS (multimeter, black probe on GND)"
- note added: "Battery voltage is NOT measured: the XIAO has 3 ADC pins only (D0..D2) and the sensors use all of them."
- note added: "D2..D7 = PL9823 (NeoPixel type, 800 kHz, 24 bit per LED): D2-D4 left side (rear -> front), D5-D7 right side"
- note added: "GPIO15 = yellow user LED on the XIAO (on = 0), a 2nd indicator for free. BOOT / RESET buttons are on the XIAO."
- note added: "GPIO16 (TX) / GPIO17 (RX) pull-up after reset + boot log / UART REPL -> no button and no motor input there."
- note added: "IN1/IN2 -> OUT1/OUT2 = LEFT motor, IN3/IN4 -> OUT3/OUT4 = RIGHT motor (+ = OUT4)"
- note added: "IR (LED_K): about 0.1 V while the IR LEDs are on (robot.sensors.leds(True)), about 2 V when off."
- note added: "IR LED: (3.3V - 1.2V - 0.1V) / 100 ohm = about 20 mA each. Q1 switches all LEDs (ambient light cancel). Photo transistor: 10k pull-up -> white = low voltage, black = high voltage"
- note added: "Inside the XIAO: 5V pin -> Schottky -> buck regulator -> 3V3 (3V3 stays up while VBAT > about 4 V)."
- note added: "Linetracer2 Lite rev.L3 : XIAO ESP32C6 on pin headers, 3 x LBR-127HLD, 1 button, 1 buzzer, 6 RGB LEDs"
- note added: "MECHANICAL: H1-H4 = gearbox frame M3 (x30/x70, y62/y96), H5 = front ball caster / skid, snap-in (x50, y11: behind the centre sensor)"
- note added: "Never solder a Li-ion cell to the XIAO's BAT pads on this robot (AA cells are on the 5V pin)."
- note added: "On pin headers the XIAO sits 2.5 mm above the board: its bare bottom test pads can not touch the tracks."
- note added: "PS1 = LEFT -> D2 (GPIO2/ADC), PS2 = CENTRE -> D1 (GPIO1/ADC), PS3 = RIGHT -> D0 (GPIO0/ADC) (seen from above, robot moving up the page)"
- note added: "Power: AA x3 (alkaline 4.5V recommended / NiMH 3.6V) -> VBAT (motors) ; VBAT -> D1 Schottky -> VSYS -> XIAO 5V pin. USB 5V can not back-feed the batteries. Never use 4 cells (the XIAO's 5V input clamps above about 6 V)."
- note added: "Q1: all IR LEDs on when SENS_LED_EN = 1 (about 60 mA)"
- note added: "Reset state (ESP32-C6 datasheet): GPIO18-23 weak pull-up during reset, then floating;"
- note added: "The body is 5.6 mm tall: the front of the robot is lifted by the 7.5 mm ball caster or skid (lens about 2.25 mm above the floor)"
- note added: "The buzzer shares D4 with the START button (no free XIAO pin). A piezo passes no DC, so reading the"
- note added: "VBAT (D1 anode / J1 +) 3.6-4.8 V, VSYS = VBAT - 0.3 V (USB: 5 V), 3V3 = 3.3 V. S1-S3: white low, black ~3 V."
- note added: "XIAO 5V pin = USB VBUS: an external supply needs a diode (D1), otherwise USB 5V charges the AA cells."
- note added: "button (input + pull-up) works; to beep, D4 becomes a PWM output - it also sounds while START is held."
- note added: "internal pull-up, pressed = 0. R10: if START is pressed while D4 beeps, only 3.3 mA flows"
- note removed: "2. MCU Raspberry Pi Pico / Pico 2 (soldered flat, no pin headers)"
- note removed: "4. BUTTON / LED"
- note removed: "5. EXPANSION (holes only)"
- note removed: "6. LINE SENSORS 3 x LBR-123F (mount on the BOTTOM side, lens to the floor, 2-3 mm gap), 12 mm apart"
- note removed: "Battery voltage: no divider on this board. The Pico measures VSYS/3 on GP29 (ADC3) internally;"
- note removed: "GP25 = on-board LED (a 2nd indicator for free). GP29/ADC3 = VSYS/3, GP24 = VBUS sense (inside Pico)."
- note removed: "IN1/IN2 -> OUT1/OUT2 = LEFT motor, IN3/IN4 -> OUT3/OUT4 = RIGHT motor"
- note removed: "IR LED: (3.3V - 1.25V) / 100 ohm = about 19 mA each. Q1 switches all LEDs (ambient light cancel). Photo transistor: 10k pull-up -> white = low voltage, black = high voltage"
- note removed: "Linetracer2 Lite : low-cost version (Pico without pin headers, 3 sensors, 1 button, 1 LED)"
- note removed: "MECHANICAL: H1-H4 = gearbox frame M3 (x30/x70, y62/y96), H5 = front skid M3 (x50, y11: behind the centre sensor)"
- note removed: "PS1 = LEFT -> GP28/ADC2, PS2 = CENTRE -> GP27/ADC1, PS3 = RIGHT -> GP26/ADC0 (seen from above, robot moving up the page)"
- note removed: "Pico W / Pico 2 W: GP29 and GP25 belong to the radio chip -> battery reading does not work, not recommended."
- note removed: "Power: AA x3 (alkaline 4.5V / NiMH 3.6V) -> VBAT (motors) ; VBAT -> D1 Schottky -> VSYS (Pico). USB 5V can not back-feed the batteries. Never use 4 cells (Pico VSYS max 5.5V)."
- note removed: "Q1: all IR LEDs on when SENS_LED_EN = 1 (about 57 mA)"
- note removed: "VBAT = VSYS + about 0.3 V (D1). GP24 = 1 while USB is plugged in."
- note removed: "internal pull-up, pressed = 0"
- note removed: "no buzzer, no power LED on the Lite board"
- title: Linetracer2 Lite - low-cost kids line tracer -> Linetracer2 Lite rev.L3 - XIAO ESP32C6 kids line tracer

Commit message: Lite rev.L3 の回路図: 文字や枠の重なりを直した（つながりは変えていない）
- テストパッドの枠と説明を右下の表題欄の上に出した（パッドを 1 列に、説明は 4 行に分けた）
- 枠 3・4・6 が図枠の右にはみ出していたのを 406.4 mm までにした。電源の枠は説明の文字が入る幅に広げた
- フルカラー LED のシンボルを 12.7 mm 角にして、中のピン名と LED の絵・RGB の字が重ならないようにした
- LED の説明が GND 記号に重なっていた → LED の列を上へ、説明を下へ。ブザーの説明はブザーの右に置いた
- R10 と START ボタンの BTN ラベル 2 つが重なっていた → 1 本の線とラベル 1 つに
- U2 の LARGE / MODE の GND 記号の字が MOT_STBY に重なっていた → 2 本をつないで GND 記号 1 つに
- J1 の部品名と VBAT の PWR_FLAG、LBR-127HLD の部品名と GND、Q1 の部品名と枠の重なりを直した
- テストパッドの「~3 V」が「-3 V」に見えていた → 「about 3 V」

ネットリストは前と同じ（32 ネット、43 部品）、ERC 0。基板・Gerber・部品表は変わらない。

Co-Authored-By: Claude Opus 5.5 <noreply@anthropic.com>
Other:
- note added: "A piezo passes no DC, so reading the button (input + pull-up)"
- note added: "IR (LED_K): about 0.1 V while the IR LEDs are on (robot.sensors.leds(True)),"
- note added: "S1-S3: white low, black about 3 V."
- note added: "START is held."
- note added: "The buzzer shares D4 with the START button (no free XIAO pin)."
- note added: "VBAT (D1 anode / J1 +) 3.6-4.8 V, VSYS = VBAT - 0.3 V (USB: 5 V), 3V3 = 3.3 V."
- note added: "about 2 V when off."
- note added: "works; to beep, D4 becomes a PWM output - it also sounds while"
- note removed: "IR (LED_K): about 0.1 V while the IR LEDs are on (robot.sensors.leds(True)), about 2 V when off."
- note removed: "The buzzer shares D4 with the START button (no free XIAO pin). A piezo passes no DC, so reading the"
- note removed: "VBAT (D1 anode / J1 +) 3.6-4.8 V, VSYS = VBAT - 0.3 V (USB: 5 V), 3V3 = 3.3 V. S1-S3: white low, black ~3 V."
- note removed: "button (input + pull-up) works; to beep, D4 becomes a PWM output - it also sounds while START is held."
- moved on the sheet: BZ1, D2, D3, D4, D5, D6, D7, Q1, R10, R7, R9, SW1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
